Commit message: Ready for Turtlebot3_Navigation Repository

File: turtlebot3_description/urdf/turtlebot3_burger.gazebo.xacro (robot description, xacro)
@@ -72,5 +72,5 @@
       <serviceName>imu_service</serviceName>
       <gaussianNoise>0.0</gaussianNoise>
-      <updateRate>0</updateRate>
+      <updateRate>200</updateRate>
       <imu>
         <noise>
@@ -101,8 +101,8 @@
         <scan>
           <horizontal>
-            <samples>360</samples>
+            <samples>720</samples>
             <resolution>1</resolution>
-            <min_angle>0.0</min_angle>
-            <max_angle>6.28319</max_angle>
+            <min_angle>-3.1416</min_angle>
+            <max_angle>3.1416</max_angle>
           </horizontal>
         </scan>

File: turtlebot3_description/urdf/turtlebot3_burger.urdf.xacro (robot description, xacro)
@@ -13,5 +13,5 @@
       <origin xyz="-0.032 0 0.0" rpy="0 0 0"/>
       <geometry>
-        <mesh filename="package://turtlebot3_description/meshes/bases/burger_base.stl" scale="0.001 0.001 0.001"/>
+        <mesh filename="package://turtlebot3_description/meshes/bases/burger_base.dae" scale="0.001 0.001 0.001"/>
       </geometry>
       <material name="light_black"/>
@@ -41,5 +41,5 @@
       <origin xyz="0 0 0" rpy="1.57 0 0"/>
       <geometry>
-        <mesh filename="package://turtlebot3_description/meshes/wheels/left_tire.stl" scale="0.001 0.001 0.001"/>
+        <mesh filename="package://turtlebot3_description/meshes/wheels/left_tire.dae" scale="0.001 0.001 0.001"/>
       </geometry>
       <material name="dark"/>
@@ -69,5 +69,5 @@
       <origin xyz="0 0 0" rpy="1.57 0 0"/>
       <geometry>
-        <mesh filename="package://turtlebot3_description/meshes/wheels/right_tire.stl" scale="0.001 0.001 0.001"/>
+        <mesh filename="package://turtlebot3_description/meshes/wheels/right_tire.dae" scale="0.001 0.001 0.001"/>
       </geometry>
       <material name="dark"/>
@@ -122,5 +122,5 @@
       <origin xyz="0 0 0.0" rpy="0 0 0"/>
       <geometry>
-        <mesh filename="package://turtlebot3_description/meshes/sensors/lds.stl" scale="0.001 0.001 0.001"/>
+        <mesh filename="package://turtlebot3_description/meshes/sensors/lds.dae" scale="0.001 0.001 0.001"/>
       </geometry>
       <material name="dark"/>
@@ -140,3 +140,87 @@
     </inertial>
   </link>
+    <!-- Camera -->
+  <link name="camera_link">
+        <visual>
+            <geometry>
+            <mesh filename="package://turtlebot3_description/meshes/sensors/rpi_camera_v2_short.dae"/>
+            </geometry>
+            <material name="camera_link_material">
+            <color rgba="0.8 0.8 0.8 1.0"/>
+            </material>
+        </visual>
+        <collision>
+            <geometry>
+            <mesh filename="package://turtlebot3_description/meshes/sensors/rpi_camera_v2_short.stl"/>
+            </geometry>
+        </collision>
+        <inertial>
+            <origin xyz="2.88715e-05 0.00248607 0.00813026" rpy="0 0 0"/>
+            <mass value="0.00217711"/>
+            <inertia ixx="2.12383e-07" ixy="6.03294e-10"  ixz="3.97667e-10" iyy="2.0411e-07" iyz="-1.46626e-09" izz="1.04162e-07" />
+        </inertial>
+    </link>
+    <joint name="chassis_1_camera_link_fixing" type="fixed">
+        <origin xyz="0.05 0.0 0.1" rpy="-1.57 0 0" />
+        <parent link="base_link" />
+        <child link="camera_link" />
+        <axis xyz="0 0 0"/>
+    </joint>
+    <link name="camera_link_frame">
+        <!-- Inertial for gazebo to take it into account, Put 1gr weight -->
+        <inertial>
+            <origin xyz="0 0 0" rpy="0 0 0"/>
+            <mass value="0.001" />
+            <inertia ixx="9.1875e-09" ixy="0.0" ixz="0.0" iyy="9.1875e-09" iyz="0.0" izz="1.378125e-08"/>
+        </inertial>
+        <visual>
+            <origin rpy="0.0 0 0" xyz="0 0 0"/>
+            <geometry>
+                <box size="0.0010 0.0005 0.0005"/>
+            </geometry>
+            <material name="green"/>
+        </visual>
+    </link>
+    <gazebo reference="camera_link_frame">
+        <material>Gazebo/Green</material>
+    </gazebo>
+    <joint name="camera_frame_joint" type="fixed">
+        <origin xyz="0.01 0.000001 0.002402" rpy="1.52 0 0" />
+        <parent link="camera_link" />
+        <child link="camera_link_frame" />
+        <axis xyz="0 0 0"/>
+    </joint>
+    <gazebo reference="camera_link_frame">
+        <sensor type="camera" name="cam">
+        <update_rate>10.0</update_rate>
+        <camera name="raspv2">
+            <pose>0 0 0 0 0 0</pose>
+            <horizontal_fov>1.3962634</horizontal_fov>
+            <image>
+            <width>640</width>
+            <height>480</height>
+            <format>R8G8B8</format>
+            </image>
+            <clip>
+                <near>0.005</near>
+                <far>20.0</far>
+            </clip>
+        </camera>
+        <plugin name="camera_controller" filename="libgazebo_ros_camera.so">
+            <alwaysOn>true</alwaysOn>
+            <updateRate>0.0</updateRate>
+            <cameraName>cv_camera</cameraName>
+            <imageTopicName>image_raw</imageTopicName>
+            <cameraInfoTopicName>camera_info</cameraInfoTopicName>
+            <frameName>camera_link_frame</frameName>
+            <hackBaseline>0.07</hackBaseline>
+            <distortionK1>0.0</distortionK1>
+            <distortionK2>0.0</distortionK2>
+            <distortionK3>0.0</distortionK3>
+            <distortionT1>0.0</distortionT1>
+            <distortionT2>0.0</distortionT2>
+        </plugin>
+        </sensor>
+    </gazebo>
 </robot>
+</robot>
